File: PCB/klor1_3/klor1_3.kicad_pcb (KiCad board)
At the start: 2 copper layers, 160 x 118.2 mm, 89 parts, among them J1 MJ-4PP-9, J2 Haptic Buzz, J3 lv27, SW1 SW_PUSH-MX_W_LED, SW10 SW_PUSH-MX_W_LED, SW11 SW_PUSH-MX_W_LED, SW12 SW_PUSH-MX_W_LED, SW13 SW_PUSH-MX_W_LED, SW14 SW_PUSH-MX_W_LED, SW15 SW_PUSH-MX_W_LED, SW16 SW_PUSH-MX_W_LED, SW17 SW_PUSH-MX_W_LED, SW18 RotaryEncoder_Switch, SW19 SW_PUSH-MX_W_LED, SW2 SW_PUSH-MX_W_LED, SW20 SW_PUSH-MX_W_LED, SW21 SW_PUSH-MX_W_LED, SW22 SW_PUSH-MX_W_LED, SW3 SW_PUSH-MX_W_LED, SW4 SW_PUSH-MX_W_LED, SW5 SW_PUSH-MX_W_LED, SW6 SW_PUSH-MX_W_LED, SW7 SW_PUSH-MX_W_LED, SW8 SW_PUSH-MX_W_LED, SW9 SW_PUSH-MX_W_LED, U1 ProMicro

Commit message: WIP: simple version
Parts:
- removed BT1: JST Connector, KLOR:JST_PH_reversible
- removed BT2: Battery_Cell, KLOR:custombatteryconnector_small
- removed BZ1: Buzzer, KLOR:Buzzer_Mallory_AST1109MLTRQ_reversible
- removed J1: MJ-4PP-9, KLOR:MJ-4PP-9
- removed J3: lv27, KLOR:lvc27_onlyInput
- removed JP1, JP16, JP17, JP18, JP19, JP2, JP20, JP21, JP22, JP23, JP24, JP25, JP26, JP27, JP28, JP3, JP4, JP5, JP6, JP7, JP8: Device_Jumper_NO_Small, KLOR:Jumper
- removed JP12, JP14: VCC Jumper, KLOR:Jumper
- removed JP13, JP15: GND Jumper, KLOR:Jumper
- removed OLED1: SSD1306, KLOR:SSD1306_128x64OLED
- removed PSW1: SW_DPDT_x2, KLOR:MSK12C02_reversible
- removed REF**: Tenting Puck, KLOR:SplitkbTentingPuckWithoutCenterHole
- added C1: 100n, KLOR:SMD-0603, F.Cu at (72.4, 98.4)
- added C2: 100n, KLOR:SMD-0603, F.Cu at (72.4, 100.9)
- added D23: D_Zener, KLOR:D_SOD-123, F.Cu at (112.6, 59.2)
- added D24: D_Zener, KLOR:D_SOD-123, F.Cu at (115.6, 59.2)
- added D25: D_Zener, KLOR:D_SOD-123, F.Cu at (118.7, 59.2)
- added D26: D_Zener, KLOR:D_SOD-123, F.Cu at (122.0, 59.2)
- added D27: D_Zener, KLOR:D_SOD-123, F.Cu at (125.3, 59.2)
- added D28: D_Zener, KLOR:D_SOD-123, F.Cu at (106.3, 101.1)
- added D29: D_Zener, KLOR:D_SOD-123, F.Cu at (106.3, 88.9)
- added D30: D_Zener, KLOR:D_SOD-123, F.Cu at (106.3, 92.0)
- added D31: D_Zener, KLOR:D_SOD-123, F.Cu at (106.3, 95.0)
- added D32: D_Zener, KLOR:D_SOD-123, F.Cu at (106.3, 98.1)
- added H1: TentingPuck, KLOR:SplitkbTentingPuckWithoutCenterHole, F.Cu at (149.6, 96.4)
- added R1: 10k, KLOR:SMD-0603, F.Cu at (84.9, 116.5)
- added R2: 10k, KLOR:SMD-0603, F.Cu at (72.4, 106.0)
- added R3: 10k, KLOR:SMD-0603, F.Cu at (72.4, 108.5)
- added R4: 10k, KLOR:SMD-0603, F.Cu at (72.4, 111.0)
- added R5: 10k, KLOR:SMD-0603, F.Cu at (95.9, 88.7)
- added R6: 10k, KLOR:SMD-0603, F.Cu at (93.3, 91.5)
- added U2: USBLC6-2SC6, Package_TO_SOT_SMD:SOT-23-6, F.Cu at (95.7, 126.0)
- D1, D10, D11, D12, D13, D14, D15, D16, D17, D18, D19, D2, D20, D21, D22, D3, D4, D5, D6, D7, D8, D9: footprint KLOR:Diode_SOD123 -> KLOR:D_SOD-123
- J2: value Haptic Buzz -> USB_C_Receptacle_USB2.0; footprint KLOR:Pimoroni Haptic Buzz DRV2605L Driver -> KLOR:USB_C_Receptacle_MUP_U22401; moved to F.Cu
- RSW1: footprint KLOR:SW_Push_1P1T-MP_NO_Horizontal_Alps_SKRTLAE010_both_sides -> KLOR:SMD_Tacticle_Switch_TS24CA_flipable
- SW1, SW10, SW11, SW12, SW13, SW14, SW15, SW16, SW17, SW19, SW2, SW20, SW21, SW22, SW3, SW4, SW5, SW6, SW7, SW8, SW9: footprint KLOR:SK6812MINI_and_cherry -> KLOR:MX_KAILH_SOCKET_1U
- SW18: value RotaryEncoder_Switch -> ALPS EC11
- moved J2 129.6 mm to (84.7, 125.1), turned to -90 degrees
- moved RSW1 68.3 mm to (97.0, 54.0), turned to 0 degrees
- moved D16 15.1 mm to (205.1, 126.5), turned to -100 degrees
- moved D2 14.4 mm to (149.7, 72.8), turned to 90 degrees
- moved D1 14.1 mm to (130.7, 76.5), turned to 90 degrees
- moved D9 14.0 mm to (188.6, 97.8), turned to 86 degrees
- moved D12 13.9 mm to (130.7, 117.6), turned to 90 degrees
- moved D5 13.9 mm to (210.7, 94.0), turned to 80 degrees
- moved D10 13.9 mm to (207.4, 112.8), turned to 80 degrees
- moved D4 13.9 mm to (189.8, 78.5), turned to 86 degrees
- moved D6 13.7 mm to (130.7, 100.4), turned to 90 degrees
- moved D3 13.7 mm to (168.8, 67.6), turned to 90 degrees
- moved D14 13.5 mm to (168.5, 105.6), turned to 90 degrees
- moved D7 12.7 mm to (149.7, 95.3), turned to 90 degrees
- moved D15 12.7 mm to (187.3, 116.6), turned to 86 degrees
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Connections:
- D1 pad 2: Net-(D1-Pad2) -> Net-(D1-A)
- D10 pad 2: Net-(D10-Pad2) -> Net-(D10-A)
- D11 pad 2: Net-(D11-Pad2) -> Net-(D11-A)
- D12 pad 2: Net-(D12-Pad2) -> Net-(D12-A)
- D13 pad 2: Net-(D13-Pad2) -> Net-(D13-A)
- D14 pad 2: Net-(D14-Pad2) -> Net-(D14-A)
- D15 pad 2: Net-(D15-Pad2) -> Net-(D15-A)
- D16 pad 2: Net-(D16-Pad2) -> Net-(D16-A)
- D17 pad 2: Net-(D17-Pad2) -> Net-(D17-A)
- D19 pad 2: Net-(D19-Pad2) -> Net-(D19-A)
- D2 pad 2: Net-(D2-Pad2) -> Net-(D2-A)
- D20 pad 2: Net-(D20-Pad2) -> Net-(D20-A)
- D21 pad 2: Net-(D21-Pad2) -> Net-(D21-A)
- D22 pad 2: Net-(D22-Pad2) -> Net-(D22-A)
- D3 pad 2: Net-(D3-Pad2) -> Net-(D3-A)
- D4 pad 2: Net-(D4-Pad2) -> Net-(D4-A)
- D5 pad 2: Net-(D5-Pad2) -> Net-(D5-A)
- D6 pad 2: Net-(D6-Pad2) -> Net-(D6-A)
- D7 pad 2: Net-(D7-Pad2) -> Net-(D7-A)
- D8 pad 2: Net-(D8-Pad2) -> Net-(D8-A)
- D9 pad 2: Net-(D9-Pad2) -> Net-(D9-A)
- SW1 pad 1: Net-(SW1-Pad1) -> Net-(D1-A)
- SW1 pad 2: GND -> SW18A
- SW10 pad 1: Net-(SW10-Pad1) -> Net-(D10-A)
- SW10 pad 2: GND -> col1
- SW11 pad 1: Net-(SW11-Pad1) -> Net-(D11-A)
- SW11 pad 2: GND -> col0
- SW12 pad 1: Net-(SW12-Pad1) -> Net-(D12-A)
- SW12 pad 2: GND -> SW18A
- SW13 pad 1: Net-(SW13-Pad1) -> Net-(D13-A)
- SW13 pad 2: GND -> col4
- SW14 pad 1: Net-(SW14-Pad1) -> Net-(D14-A)
- SW14 pad 2: GND -> col3
- SW15 pad 1: Net-(SW15-Pad1) -> Net-(D15-A)
- SW15 pad 2: GND -> col2
- SW16 pad 1: Net-(SW10-Pad3) -> Net-(D16-A)
- SW16 pad 2: GND -> col1
- SW17 pad 1: unconnected-(SW17-Pad1) -> Net-(D17-A)
- SW17 pad 2: GND -> col0
- SW18 pad A: ENCA -> Net-(C2-Pad1)
- SW18 pad B: ENCB -> Net-(C1-Pad1)
- SW18 pad S1: col5 -> SW18A
- SW18 pad S2: SW18B -> Col5
- SW19 pad 1: Net-(JP26-Pad1) -> Net-(D19-A)
- SW19 pad 2: GND -> col4
- SW2 pad 1: Net-(SW2-Pad1) -> Net-(D2-A)
- SW2 pad 2: GND -> col4
- SW20 pad 1: Net-(SW20-Pad1) -> Net-(D20-A)
- SW20 pad 2: GND -> col3
- SW21 pad 1: Net-(SW12-Pad3) -> Net-(D21-A)
- SW21 pad 2: GND -> col2
- SW22 pad 1: Net-(SW14-Pad3) -> Net-(D22-A)
- SW22 pad 2: GND -> col1
- SW3 pad 1: Net-(SW3-Pad1) -> Net-(D3-A)
- SW3 pad 2: GND -> col3
- SW4 pad 1: Net-(SW4-Pad1) -> Net-(D4-A)
- SW4 pad 2: GND -> col2
- SW5 pad 1: Net-(SW11-Pad3) -> Net-(D5-A)
- SW5 pad 2: GND -> col1
- SW6 pad 1: Net-(SW1-Pad3) -> Net-(D6-A)
- SW6 pad 2: GND -> SW18A
- SW7 pad 1: Net-(SW13-Pad3) -> Net-(D7-A)
- SW7 pad 2: GND -> col4
- SW8 pad 1: Net-(SW3-Pad3) -> Net-(D8-A)
- SW8 pad 2: GND -> col3
- SW9 pad 1: Net-(SW15-Pad3) -> Net-(D9-A)
- SW9 pad 2: GND -> col2
- U1 pad 1: LED -> TX_ESD
- U1 pad 12: AUDIO -> handness
- U1 pad 13: col5 -> SW18A
- U1 pad 2: TX -> RX_ESD
- U1 pad 24: +BATT -> VBUS
- U1 pad 5: SDA -> unconnected-(U1-2/D1/SDA-Pad5)
- U1 pad 6: SCL -> unconnected-(U1-3/D0/SCL-Pad6)
- U1 pad 7: RX -> unconnected-(U1-4/D4-Pad7)
Routing:
- net VCC: track 780.6 -> 14.4 mm, vias 32 -> 0
- net SDA: track 277.8 -> 0.00 mm, vias 5 -> 0
- net SCL: track 266.4 -> 0.00 mm, vias 4 -> 0
- net col4: track 348.7 -> 180.9 mm, vias 7 -> 2
- net col5: track 143.9 -> 0.00 mm, vias 6 -> 0
- net col3: track 336.4 -> 199.1 mm, vias 7 -> 2
- net LED: track 131.4 -> 0.00 mm, vias 4 -> 0
- net col2: track 333.2 -> 225.3 mm, vias 7 -> 2
- net TX: track 102.6 -> 0.00 mm, vias 2 -> 0
- net AUDIO: track 101.9 -> 0.00 mm
- net RX: track 87.5 -> 0.00 mm, vias 2 -> 0
- net RESET: track 77.9 -> 14.4 mm, vias 2 -> 1
- net col1: track 310.8 -> 250.3 mm, vias 6 -> 2
- net /PSW: track 59.2 -> 0.00 mm, vias 2 -> 0
- net SW18A: track 0.00 -> 57.7 mm, vias 0 -> 3
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Other:
- outline, holes or cut-outs redrawn
- board text added: "--HAND"
- board text added: "REVISION SIMPLE BY KARLK90"
- board text added: "VBUS--"
- board text removed: "--AUDIO"
- board text removed: "--LED"
- board text removed: "--SCL"
- board text removed: "--SDA"
- board text removed: "BATT"
- board text removed: "BATT+--"
- board text removed: "BLK"
- board text removed: "BUZZER"
- board text removed: "GND"
- board text removed: "HAPTIC BUZZ"
- board text removed: "OLED"
- board text removed: "RED"
- board text removed: "REVISION 1.3 BY GEIST"
- board text removed: "SCL"
- board text removed: "SDA"
- board text removed: "TENTING PUCK"
- board text removed: "TRACK BALL"
- board text removed: "VCC"
