File: PCB/klor1_3/klor1_3.kicad_pcb (KiCad board)
At the start: 2 copper layers, 160 x 118.2 mm, 76 parts, among them J2 USB_C_Receptacle_USB2.0, SW1 SW_PUSH-MX_W_LED, SW10 SW_PUSH-MX_W_LED, SW11 SW_PUSH-MX_W_LED, SW12 SW_PUSH-MX_W_LED, SW13 SW_PUSH-MX_W_LED, SW14 SW_PUSH-MX_W_LED, SW15 SW_PUSH-MX_W_LED, SW16 SW_PUSH-MX_W_LED, SW17 SW_PUSH-MX_W_LED, SW18 ALPS EC11, SW19 SW_PUSH-MX_W_LED, SW2 SW_PUSH-MX_W_LED, SW20 SW_PUSH-MX_W_LED, SW21 SW_PUSH-MX_W_LED, SW22 SW_PUSH-MX_W_LED, SW3 SW_PUSH-MX_W_LED, SW4 SW_PUSH-MX_W_LED, SW5 SW_PUSH-MX_W_LED, SW6 SW_PUSH-MX_W_LED, SW7 SW_PUSH-MX_W_LED, SW8 SW_PUSH-MX_W_LED, SW9 SW_PUSH-MX_W_LED, U1 ProMicro, U2 USBLC6-2SC6

Commit message: wip
Parts:
- added C3: 100n, KLOR:SMD-0603, F.Cu at (93.6, 127.7)
- added D33: D_Zener, KLOR:D_SOD-123, F.Cu at (96.7, 103.7)
- added D34: D_Zener, KLOR:D_SOD-123, F.Cu at (93.7, 103.7)
- added R10: 10k, KLOR:SMD-0603, F.Cu at (108.9, 77.5)
- added R11: 10k, KLOR:SMD-0603, F.Cu at (108.9, 81.4)
- added R12: 10k, KLOR:SMD-0603, F.Cu at (108.9, 85.4)
- added R13: 10k, KLOR:SMD-0603, F.Cu at (108.9, 71.6)
- added R14: 10k, KLOR:SMD-0603, F.Cu at (108.9, 75.5)
- added R15: 10k, KLOR:SMD-0603, F.Cu at (108.9, 79.5)
- added R16: 10k, KLOR:SMD-0603, F.Cu at (108.9, 83.4)
- added R7: 10k, KLOR:SMD-0603, F.Cu at (108.9, 67.6)
- added R8: 10k, KLOR:SMD-0603, F.Cu at (108.9, 69.6)
- added R9: 10k, KLOR:SMD-0603, F.Cu at (108.9, 73.5)
- moved D28 42.1 mm to (112.6, 59.5), turned to 90 degrees
- moved C1 31.6 mm to (103.6, 103.7), turned to 90 degrees
- moved R2 29.2 mm to (101.5, 103.7), turned to -90 degrees
- moved R4 20.2 mm to (91.2, 103.7), turned to 90 degrees
- moved R1 19.2 mm to (99.2, 103.7), turned to 90 degrees
- moved R3 17.4 mm to (89.1, 103.7), turned to -90 degrees
- moved C2 14.9 mm to (87.0, 103.7), turned to 90 degrees
- moved D18 8.90 mm to (106.5, 113.8), turned to 90 degrees
- moved R6 5.47 mm to (97.9, 88.4), turned to 90 degrees
- moved D23 3.31 mm to (115.9, 59.5)
- moved D24 3.31 mm to (118.9, 59.5)
- moved D25 3.31 mm to (122.0, 59.5)
- moved D26 3.31 mm to (125.3, 59.5)
- moved D27 3.31 mm to (128.6, 59.5)
- moved U2 1.90 mm to (94.1, 125.1)
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Connections:
- D18 pad 2: SW18B -> ENC_B
- D28 pad 1: SW18A -> col5
- SW1 pad 2: SW18A -> col5
- SW12 pad 2: SW18A -> col5
- SW18 pad S1: SW18A -> col5
- SW18 pad S2: Col5 -> ENC_B
- SW6 pad 2: SW18A -> col5
- U1 pad 10: row2 -> Net-(U1-7/E6)
- U1 pad 11: row3 -> Net-(U1-8/B4)
- U1 pad 13: SW18A -> Net-(U1-B6/10)
- U1 pad 14: col4 -> Net-(U1-B2/16)
- U1 pad 15: col3 -> Net-(U1-B3/14)
- U1 pad 16: col2 -> Net-(U1-B1/15)
- U1 pad 17: col1 -> Net-(U1-F7/A0)
- U1 pad 18: col0 -> Net-(U1-F6/A1)
- U1 pad 5: unconnected-(U1-2/D1/SDA-Pad5) -> GND
- U1 pad 6: unconnected-(U1-3/D0/SCL-Pad6) -> GND
- U1 pad 7: unconnected-(U1-4/D4-Pad7) -> GND
- U1 pad 8: row0 -> Net-(U1-5/C6)
- U1 pad 9: row1 -> Net-(U1-6/D7)
Routing:
- net VBUS: track 18.4 -> 105.5 mm, vias 0 -> 4
- net RX_ESD: track 18.2 -> 88.0 mm, vias 0 -> 2
- net TX_ESD: track 21.8 -> 89.7 mm, vias 0 -> 2
- net col5: track 0.00 -> 65.9 mm, vias 0 -> 3
- net VCC: track 14.4 -> 77.7 mm
- net SW18A: track 57.7 -> 0.00 mm, vias 3 -> 0
- net ENCA: track 14.5 -> 56.0 mm, vias 1 -> 2
- net ENCB: track 14.5 -> 51.1 mm, vias 1 -> 2
- net Net-(C1-Pad1): track 0.00 -> 26.7 mm
- net col0: track 189.3 -> 163.8 mm, vias 4 -> 3
- net col1: track 250.3 -> 225.7 mm
- net Net-(U1-5/C6): track 0.00 -> 22.5 mm
- net Net-(U1-F7/A0): track 0.00 -> 22.1 mm, vias 0 -> 1
- net col2: track 225.3 -> 203.4 mm
- net Net-(U1-F6/A1): track 0.00 -> 21.8 mm, vias 0 -> 1
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Other:
- outline, holes or cut-outs redrawn
- board text added: "HAND--"
- board text added: "REVISION SIMPLE ESD BY GEIST x KARLK90"
- board text added: "ROW0--"
- board text added: "ROW1--"
- board text added: "ROW2--"
- board text added: "ROW3--"
- board text removed: "ENC"
- board text removed: "LOST THUMB?"
- board text removed: "REVISION SIMPLE BY KARLK90"
- board text removed: "RST"
