File: PCB/klor1_3/klor1_3.kicad_sch (KiCad schematic)
At the start: 88 parts, among them J1 MJ-4PP-9, J2 Haptic Buzz, J3 lv27, SW1 SW_PUSH-MX_W_LED, SW10 SW_PUSH-MX_W_LED, SW11 SW_PUSH-MX_W_LED, SW12 SW_PUSH-MX_W_LED, SW13 SW_PUSH-MX_W_LED, SW14 SW_PUSH-MX_W_LED, SW15 SW_PUSH-MX_W_LED, SW16 SW_PUSH-MX_W_LED, SW17 SW_PUSH-MX_W_LED, SW18 RotaryEncoder_Switch, SW19 SW_PUSH-MX_W_LED, SW2 SW_PUSH-MX_W_LED, SW20 SW_PUSH-MX_W_LED, SW21 SW_PUSH-MX_W_LED, SW22 SW_PUSH-MX_W_LED, SW3 SW_PUSH-MX_W_LED, SW4 SW_PUSH-MX_W_LED, SW5 SW_PUSH-MX_W_LED, SW6 SW_PUSH-MX_W_LED, SW7 SW_PUSH-MX_W_LED, SW8 SW_PUSH-MX_W_LED, SW9 SW_PUSH-MX_W_LED, U1 ProMicro

Commit message: WIP: simple version
Parts:
- removed BT1: JST Connector, KLOR:JST_PH_reversible, symbol Device:Battery_Cell
- removed BT2: Battery_Cell, KLOR:custombatteryconnector_small, symbol Device:Battery_Cell
- removed BZ1: Buzzer, KLOR:Buzzer_Mallory_AST1109MLTRQ_reversible, symbol Device:Buzzer
- removed J1: MJ-4PP-9, KLOR:MJ-4PP-9, symbol KLORlib:MJ-4PP-9 TRRS
- removed J2: Haptic Buzz, KLOR:Pimoroni Haptic Buzz DRV2605L Driver, symbol Connector_Generic:Conn_01x05
- removed J3: lv27, KLOR:lvc27_onlyInput, symbol Connector_Generic:Conn_01x05
- removed JP1, JP16, JP17, JP18, JP19, JP2, JP21, JP22, JP23, JP24, JP25, JP26, JP27, JP28, JP3, JP4, JP5, JP6, JP7, JP8: Device_Jumper_NO_Small, KLOR:Jumper, symbol KLORlib:Device_Jumper_NO_Small
- removed JP12, JP14: VCC Jumper, KLOR:Jumper, symbol Jumper:Jumper_2_Open
- removed JP13, JP15: GND Jumper, KLOR:Jumper, symbol Jumper:Jumper_2_Open
- removed JP20: Device_Jumper_NO_Small, KLOR:Jumper, symbol SofleKeyboard-cache:Device_Jumper_NO_Small
- removed OLED1: SSD1306, KLOR:SSD1306_128x64OLED, symbol SSD1306-128x64_OLED:SSD1306
- removed PSW1: SW_DPDT_x2, KLOR:MSK12C02_reversible, symbol Switch:SW_DPDT_x2
- removed unit 2 of SW1
- removed unit 2 of SW10
- removed unit 2 of SW11
- removed unit 2 of SW12
- removed unit 2 of SW13
- removed unit 2 of SW14
- removed unit 2 of SW15
- removed unit 2 of SW16
- removed unit 2 of SW17
- removed SW18: RotaryEncoder_Switch, KLOR:RotaryEncoder_Alps_EC11E-Switch_Vertical_H20mm-keebio_modified, symbol Device:RotaryEncoder_Switch
- removed unit 2 of SW19
- removed unit 2 of SW2
- removed unit 2 of SW20
- removed unit 2 of SW21
- removed unit 2 of SW22
- removed unit 2 of SW3
- removed unit 2 of SW4
- removed unit 2 of SW5
- removed unit 2 of SW6
- removed unit 2 of SW7
- removed unit 2 of SW8
- removed unit 2 of SW9
- added C1, C2: 100n, KLOR:SMD-0603, symbol YAEMK:C
- added D23, D24, D25, D26, D27, D28, D29, D30, D31, D32: D_Zener, KLOR:D_SOD-123, symbol Device:D_Zener
- added H1: TentingPuck, KLOR:SplitkbTentingPuckWithoutCenterHole, symbol Mechanical:MountingHole
- added J2: USB_C_Receptacle_USB2.0, KLOR:USB_C_Receptacle_MUP_U22401, symbol Connector:USB_C_Receptacle_USB2.0
- added R1, R2, R24, R25, R3, R4: 10k, KLOR:SMD-0603, symbol YAEMK:R
- added SW1: ALPS EC11, KLOR:RotaryEncoder_Alps_EC11E-Switch_Vertical_H20mm-keebio_modified, symbol YAEMK:Rotary_Encoder_Switch
- added U2: USBLC6-2SC6, Package_TO_SOT_SMD:SOT-23-6, symbol Power_Protection:USBLC6-2SC6
- RSW1: footprint KLOR:SW_Push_1P1T-MP_NO_Horizontal_Alps_SKRTLAE010_both_sides -> KLOR:SMD_Tacticle_Switch_TS24CA_flipable
- SW1, SW10, SW11, SW12, SW13, SW14, SW15, SW16, SW17, SW19, SW2, SW20, SW21, SW22, SW3, SW4, SW5, SW6, SW7, SW8, SW9: footprint KLOR:SK6812MINI_and_cherry -> KLOR:MX_KAILH_SOCKET_1U; symbol KLORlib:SW_PUSH-MX_W_LED -> Switch:SW_Push
Connections:
- net ENCA: now also R1.2
- net ENCB: now also R4.2
- net GND: now also C1.2, C2.2, D23.2 (A), D24.2 (A), D25.2 (A), D26.2 (A), D27.2 (A), D28.2 (A), D29.2 (A), D30.2 (A), D31.2 (A), D32.2 (A), J2.A1 (GND), J2.A12 (GND), J2.B1 (GND), J2.B12 (GND), J2.S1 (SHIELD), R25.2, SW1.C, U2.2 (GND)
- net RX: now also J2.A6 (D+), J2.B6 (D+), U2.3 (I/O2); no longer U1.7 (4/D4)
- net SW18A: now also SW1.2, SW12.2, SW6.2, D28.1 (K), SW1.S1; no longer SW1.5, SW12.5, SW6.5
- net TX: now also J2.A7 (D-), J2.B7 (D-), U2.1 (I/O1); no longer U1.2 (RX1/D2)
- net VCC: now also R2.1, R24.1, R3.1
- net col0: now also SW11.2, SW17.2, D23.1 (K); no longer SW11.5, SW17.5
- net col1: now also SW10.2, SW16.2, SW22.2, SW5.2, D24.1 (K); no longer SW10.5, SW16.5, SW22.5, SW5.5
- net col2: now also SW15.2, SW21.2, SW4.2, SW9.2, D25.1 (K); no longer SW15.5, SW21.5, SW4.5, SW9.5
- net col3: now also SW14.2, SW20.2, SW3.2, SW8.2, D26.1 (K); no longer SW14.5, SW20.5, SW3.5, SW8.5
- net col4: now also SW13.2, SW19.2, SW2.2, SW7.2, D27.1 (K); no longer SW13.5, SW19.5, SW2.5, SW7.5
- net row0: now also D29.1 (K)
- net row1: now also D30.1 (K)
- net row2: now also D31.1 (K)
- net row3: now also D32.1 (K)
- net at D3.2 (A): now also SW3.1; no longer SW3.6
- net at D14.2 (A): now also SW14.1; no longer SW14.6
- net at D13.2 (A): now also SW13.1; no longer SW13.6
- net at D16.2 (A): now also SW16.1; no longer SW16.6
- net at D20.2 (A): now also SW20.1; no longer SW20.6
- net at D19.2 (A): now also SW19.1; no longer SW19.6
- net at D9.2 (A): now also SW9.1; no longer SW9.6
- net at D15.2 (A): now also SW15.1; no longer SW15.6
- net at D4.2 (A): now also SW4.1; no longer SW4.6
- net at D7.2 (A): now also SW7.1; no longer SW7.6
- net at D6.2 (A): now also SW6.1; no longer SW6.6
- net at D1.2 (A): now also SW1.1; no longer SW1.6
- net at D5.2 (A): now also SW5.1; no longer SW5.6
- net at D21.2 (A): now also SW21.1; no longer SW21.6
- net at D2.2 (A): now also SW2.1; no longer SW2.6
- net at D17.2 (A): now also SW17.1; no longer SW17.6
- net at D12.2 (A): now also SW12.1; no longer SW12.6
- net at D10.2 (A): now also SW10.1; no longer SW10.6
- net at D11.2 (A): now also SW11.1; no longer SW11.6
- net at D8.2 (A): now also SW8.1; no longer SW8.6
- net at D22.2 (A): now also SW22.1; no longer SW22.6
- net +BATT renamed VBUS
- net VBUS: now also J2.A4 (VBUS), J2.A9 (VBUS), J2.B4 (VBUS), J2.B9 (VBUS), U2.5 (VBUS)
- net AUDIO renamed handness
- net handness: now also R24.2, R25.1
- net LED renamed TX_ESD
- net TX_ESD: now also U2.6 (I/O1)
- net SCL: no longer names the net of U1.6 (3/D0/SCL)
- net SDA: no longer names the net of U1.5 (2/D1/SDA)
- new net: C1.1, R1.1, R2.2, SW1.B
- new net: C2.1, R3.2, R4.1, SW1.A
- new net Col5: SW1.S2
- new net RX_ESD: U1.2 (RX1/D2), U2.4 (I/O2)
- no-connect marks 2 -> 7
Other:
- note added: "Populate R5 when board is the left side. Populate R6 when board is the right side."
- note removed: "HAPTIC FEEDBACK"
- note removed: "LED MATRIX"
- note removed: "OLED"
- note removed: "ON/OFF SWITCH BATTERY"
- note removed: "SPEAKER"
- note removed: "TRACKBALL MODULE"
