File: PCB/klor1_3/klor1_3.kicad_sch (KiCad schematic)
At the start: 76 parts, among them J2 USB_C_Receptacle_USB2.0, SW1 ALPS EC11, SW1 SW_PUSH-MX_W_LED, SW10 SW_PUSH-MX_W_LED, SW11 SW_PUSH-MX_W_LED, SW12 SW_PUSH-MX_W_LED, SW13 SW_PUSH-MX_W_LED, SW14 SW_PUSH-MX_W_LED, SW15 SW_PUSH-MX_W_LED, SW16 SW_PUSH-MX_W_LED, SW17 SW_PUSH-MX_W_LED, SW19 SW_PUSH-MX_W_LED, SW2 SW_PUSH-MX_W_LED, SW20 SW_PUSH-MX_W_LED, SW21 SW_PUSH-MX_W_LED, SW22 SW_PUSH-MX_W_LED, SW3 SW_PUSH-MX_W_LED, SW4 SW_PUSH-MX_W_LED, SW5 SW_PUSH-MX_W_LED, SW6 SW_PUSH-MX_W_LED, SW7 SW_PUSH-MX_W_LED, SW8 SW_PUSH-MX_W_LED, SW9 SW_PUSH-MX_W_LED, U1 ProMicro, U2 USBLC6-2SC6

Commit message: wip
Parts:
- added C1: 100n, KLOR:SMD-0603, symbol YAEMK:C
- added D33, D34: D_Zener, KLOR:D_SOD-123, symbol Device:D_Zener
- added R4 (x10): 10k, KLOR:SMD-0603, symbol YAEMK:R
Connections:
- net SW18B is gone; now on net ENC_B: D18.2 (A)
- net ENCA: now also D33.1 (K)
- net ENCB: now also D34.1 (K)
- net GND: now also U1.5 (2/D1/SDA), U1.6 (3/D0/SCL), U1.7 (4/D4), C1.2, D33.2 (A), D34.2 (A)
- net VBUS: now also C1.1
- net col0: now also R4.2; no longer U1.18 (F6/A1)
- net col1: now also R4.2; no longer U1.17 (F7/A0)
- net col2: now also R4.2; no longer U1.16 (B1/15)
- net col3: now also R4.2; no longer U1.15 (B3/14)
- net col4: now also R4.2; no longer U1.14 (B2/16)
- net row0: now also R4.1; no longer U1.8 (5/C6)
- net row1: now also R4.1; no longer U1.9 (6/D7)
- net row2: now also R4.1; no longer U1.10 (7/E6)
- net row3: now also R4.1; no longer U1.11 (8/B4)
- net Col5 renamed ENC_B
- net SW18A renamed col5
- net col5: now also R4.2; no longer U1.13 (B6/10)
- new net: R4.1, U1.18 (F6/A1)
- new net: R4.1, U1.14 (B2/16)
- new net: R4.1, U1.16 (B1/15)
- new net: R4.2, U1.11 (8/B4)
- new net: R4.1, U1.17 (F7/A0)
- new net: R4.1, U1.13 (B6/10)
- new net: R4.2, U1.8 (5/C6)
- new net: R4.1, U1.15 (B3/14)
- new net: R4.2, U1.9 (6/D7)
- new net: R4.2, U1.10 (7/E6)
- no-connect marks 7 -> 4
Other:
- moved on the sheet: H1, MH1, MH2, MH3, MH4, MH5, MH6, MH7, MH8, MH9, R24, R25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
